File: PCB/pwrbox-v0.1/pwrbox-v0.1.kicad_sch (KiCad schematic)
At the start: 33 parts, among them J1 STEMMA_I2C_QT, J2 Conn_01x01, Q1 RFP30N06LE, Q2 RFP30N06LE, Q3 RFP30N06LE, Q4 RFP30N06LE, Q5 RFP30N06LE, Q6 RFP30N06LE, U3 TCA9534

Commit message: update connectors
Parts:
- J1: footprint (none) -> Connector_JST:JST_SH_BM04B-SRSS-TB_1x04-1MP_P1.00mm_Vertical
Changed lines of the file:
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@@
     (property "Reference" "J1" (id 0) (at 128.27 22.86 0))
     (property "Value" "STEMMA_I2C_QT" (id 1) (at 128.27 25.4 0))
-    (property "Footprint" "" (id 2) (at 128.27 31.75 0)
+    (property "Footprint" "Connector_JST:JST_SH_BM04B-SRSS-TB_1x04-1MP_P1.00mm_Vertical" (id 2) (at 128.27 31.75 0)
       (effects (font (size 1.27 1.27)) hide)
     )
@@
     )
     (path "/b147ac7b-ecaa-435a-9dbb-edf7b2985e71"
-      (reference "J1") (unit 1) (value "STEMMA_I2C_QT") (footprint "")
+      (reference "J1") (unit 1) (value "STEMMA_I2C_QT") (footprint "Connector_JST:JST_SH_BM04B-SRSS-TB_1x04-1MP_P1.00mm_Vertical")
     )
     (path "/fac4a43a-8af7-4b54-b58e-40a7801daa51"
